File: elec/digit_segment.kicad_sch (KiCad schematic)
At the start: 7 parts

Commit message: Finalise PCB
Other:
- company: (none) -> Ng Chen-Xuan
- title: (none) -> USB-C PD Portable PSU
Changed lines of the file:
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@@
 	(generator_version "10.0")
 	(paper "A4")
+	(title_block
+		(title "USB-C PD Portable PSU")
+		(date "2026-06-25")
+		(rev "v1")
+		(company "Ng Chen-Xuan")
+	)
 	(junction
 		(at 138.43 106.68)
