File: elec/display.kicad_sch (KiCad schematic)
At the start: 5 parts, among them U6 IS31FL3731-QF

Commit message: Populate LCSC Params, Assign Footprints, Update STM32CubeMX
Parts:
- D58, D59: footprint (none) -> LED_SMD:LED_0603_1608Metric
- R29, R30: footprint (none) -> Resistor_SMD:R_0603_1608Metric
Changed lines of the file:
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@@
 			)
 		)
-		(property "Footprint" ""
+		(property "Footprint" "Resistor_SMD:R_0603_1608Metric"
 			(at 77.47 133.858 90)
 			(hide yes)
@@
 			)
 		)
-		(property "Footprint" ""
+		(property "Footprint" "LED_SMD:LED_0603_1608Metric"
 			(at 232.41 43.18 0)
 			(hide yes)
@@
 			)
 		)
-		(property "Footprint" ""
+		(property "Footprint" "LED_SMD:LED_0603_1608Metric"
 			(at 232.41 83.82 0)
 			(hide yes)
@@
 			)
 		)
-		(property "Footprint" ""
+		(property "Footprint" "Resistor_SMD:R_0603_1608Metric"
 			(at 77.47 149.098 90)
 			(hide yes)

Commit message: PCB layout
Parts:
- added D63, D64, D65: LED, LED_SMD:LED_0603_1608Metric, symbol Device:LED
- added R34, R35, R36: 1k, Resistor_SMD:R_0603_1608Metric, symbol Device:R
Connections:
- net GNDREF: now also D63.1 (K), D64.1 (K), D65.1 (K)
- new net: D64.2 (A), R35.2
- new net: D65.2 (A), R36.2
- new net: D63.2 (A), R34.2
- new net CC_INDICATOR: R35.1
- new net CV_INDICATOR: R34.1
- new net OCP_INDICATOR: R36.1

Commit message: Completed Routing
Connections:
- net DIG_2: now also D59.1 (K)
- net DIG_7: no longer D59.1 (K)
