File: elec/display.kicad_sch (KiCad schematic)
At the start: 11 parts, among them U6 IS31FL3731-QF

Commit message: Finalise PCB
Parts:
- added C23: 1uF, Capacitor_SMD:C_0603_1608Metric, symbol Device:C
- added C24: 0.1uF, Capacitor_SMD:C_0603_1608Metric, symbol Device:C
Connections:
- net +3V3: now also C23.1, C24.2
- net GNDREF: now also C23.2, C24.1
Other:
- company: (none) -> Ng Chen-Xuan
- title: (none) -> USB-C PD Portable PSU
