File: elec/elec.kicad_sch (KiCad schematic)
At the start: 85 parts, among them J1 USB_C_Receptacle, J2 Conn_01x05, J3 Screw_Terminal_01x02, J4 Conn_01x03, J5 Conn_01x03, Q1 AO4419, SW2 SW_Push, SW3 SW_Push, SW4 SW_Push, SW5 SW_Push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

Commit message: Finalise PCB
Parts:
- added C22: 1uF, Capacitor_SMD:C_0603_1608Metric, symbol Device:C
- added R40: 1M, Resistor_SMD:R_0603_1608Metric, symbol Device:R
- added R41: 20k, Resistor_SMD:R_0603_1608Metric, symbol Device:R
Connections:
- net +3V3: now also C22.1, R41.1
- net GNDREF: now also R6.2, C22.2, R40.2
- net USB-C_INT: now also R41.2
- net at U2.1 (FB): now also C5.2, R4.2, R5.2, R6.1; no longer R6.2
- net at U1.6 (~{DEBUG}): now also R40.1
- no-connect marks 12 -> 11
Other:
- company: (none) -> Ng Chen-Xuan
- title: (none) -> USB-C PD Portable PSU
- moved on the sheet: D1, J1, Q1, R10, R7, R8, R9, U1
